Commit message: [FEAT] Added D435i to urdf model

File: urdf/open_manipulator.urdf.xacro (robot description, xacro)
@@ -236,10 +236,14 @@
   </link>
   <!-- Realsense Camera Joint Position -->
-<!--   <joint name="camera_joint" type="fixed">
+  <joint name="realsense_camera_joint" type="fixed">
     <axis xyz="0 1 0" />
-    <origin xyz="0.070 0.032 0.052" rpy="0 0 0"/>
-    <parent link="link5"/>
-    <child link="camera_link"/>
-  </joint>
-  <link name="camera_link"/> -->
+    <origin xyz="0.06 0.0 0.039" rpy="0 0 0"/>
+    <parent link="link5"/>
+    <child link="base_link"/>
+  </joint>
+  <link name="base_link">
+  </link>
+  <xacro:sensor_d435i parent="base_link" use_nominal_extrinsics="$(arg use_nominal_extrinsics)">
+      <origin xyz="0 0 0" rpy="0 0 0"/>
+    </xacro:sensor_d435i>
 </robot>

File: urdf/open_manipulator_robot.urdf.xacro (robot description, xacro)
@@ -2,4 +2,7 @@
 <!-- Open_Manipulator Chain -->
 <robot name="open_manipulator" xmlns:xacro="http://ros.org/wiki/xacro">
+  <!-- Import RealSense D435i -->
+  <xacro:arg name="use_nominal_extrinsics" default="false" />
+  <xacro:include filename="$(find realsense2_description)/urdf/_d435i.urdf.xacro"/>
   <!-- Import Rviz colors -->
   <xacro:include filename="$(find rgbd-pepper-pose-estimation-ros)/urdf/materials.xacro" />

Commit message: [FEAT] Started dev with  fixed camera

File: urdf/open_manipulator.urdf.xacro (robot description, xacro)
@@ -2,4 +2,5 @@
 <!-- Open_Manipulator Chain -->
 <robot xmlns:xacro="http://ros.org/wiki/xacro">
+<xacro:property name="M_PI" value="3.1415926535897931" />
   <!-- Link 1 -->
   <link name="link1">
@@ -238,6 +239,6 @@
   <joint name="realsense_camera_joint" type="fixed">
     <axis xyz="0 1 0" />
-    <origin xyz="0.06 0.0 0.039" rpy="0 0 0"/>
-    <parent link="link5"/>
+    <origin xyz="0.18 -0.88 0.2" rpy="0 0 ${M_PI/2}"/>
+    <parent link="link1"/>
     <child link="base_link"/>
   </joint>
